Commit message: [ARM-54] Mise à jour des sous-modules dans un fork AltranArmada

File: rotors_description/urdf/component_snippets.xacro (robot description, xacro)
@@ -18,5 +18,5 @@
 <robot xmlns:xacro="http://ros.org/wiki/xacro">
   <!-- Macro to add logging to a bag file. -->
-  <xacro:macro name="bag_plugin_macro"
+   <xacro:macro name="bag_plugin_macro"
     params="namespace bag_file rotor_velocity_slowdown_sim">
     <gazebo>
@@ -79,5 +79,5 @@
           </clip>
           <noise>
-            <type>gaussian</type>
+          <type>gaussian</type>
             <!-- Noise is sampled independently per pixel on each frame.
                  That pixel's noise value is added to each of its color
@@ -104,5 +104,5 @@
       </sensor>
     </gazebo>
-  </xacro:macro>
+  </xacro:macro> -->
   <!-- Macro to add the controller interface. -->
   <xacro:macro name="controller_plugin_macro" params="namespace imu_sub_topic">
@@ -118,6 +118,7 @@
     </gazebo>
   </xacro:macro>
-  <!-- Macro to add an IMU. -->
-  <xacro:macro name="imu_plugin_macro"
+  <!-- Macro to add an IMU.
+-->
+   <xacro:macro name="imu_plugin_macro"
     params="namespace imu_suffix parent_link imu_topic
       mass_imu_sensor gyroscope_noise_density gyroscopoe_random_walk
@@ -127,5 +128,5 @@
       *inertia *origin">
     <!-- IMU link -->
-    <link name="${namespace}/imu${imu_suffix}_link">
+     <link name="${namespace}/imu${imu_suffix}_link">
       <inertial>
         <xacro:insert_block name="inertia" />
@@ -145,22 +146,21 @@
       <!-- A good description of the IMU parameters can be found in the kalibr documentation:
            https://github.com/ethz-asl/kalibr/wiki/IMU-Noise-Model-and-Intrinsics -->
-        <robotNamespace>${namespace}</robotNamespace> <!-- (string, required): ros namespace in which the messages are published -->
-        <linkName>${namespace}/imu${imu_suffix}_link</linkName> <!-- (string, required): name of the body which holds the IMU sensor -->
-        <imuTopic>${imu_topic}</imuTopic> <!-- (string): name of the sensor output topic and prefix of service names (defaults to imu) -->
-        <gyroscopeNoiseDensity>${gyroscope_noise_density}</gyroscopeNoiseDensity> <!-- Gyroscope noise density (two-sided spectrum) [rad/s/sqrt(Hz)] -->
-        <gyroscopeRandomWalk>${gyroscopoe_random_walk}</gyroscopeRandomWalk> <!-- Gyroscope bias random walk [rad/s/s/sqrt(Hz)] -->
-        <gyroscopeBiasCorrelationTime>${gyroscope_bias_correlation_time}</gyroscopeBiasCorrelationTime> <!-- Gyroscope bias correlation time constant [s] -->
-        <gyroscopeTurnOnBiasSigma>${gyroscope_turn_on_bias_sigma}</gyroscopeTurnOnBiasSigma> <!-- Gyroscope turn on bias standard deviation [rad/s] -->
-        <accelerometerNoiseDensity>${accelerometer_noise_density}</accelerometerNoiseDensity> <!-- Accelerometer noise density (two-sided spectrum) [m/s^2/sqrt(Hz)] -->
-        <accelerometerRandomWalk>${accelerometer_random_walk}</accelerometerRandomWalk> <!-- Accelerometer bias random walk. [m/s^2/s/sqrt(Hz)] -->
-        <accelerometerBiasCorrelationTime>${accelerometer_bias_correlation_time}</accelerometerBiasCorrelationTime> <!-- Accelerometer bias correlation time constant [s] -->
-        <accelerometerTurnOnBiasSigma>${accelerometer_turn_on_bias_sigma}</accelerometerTurnOnBiasSigma> <!-- Accelerometer turn on bias standard deviation [m/s^2] -->
-      </plugin>
+        <robotNamespace>${namespace}</robotNamespace>  <!-- (string, required): ros namespace in which the messages are published -->
+         <linkName>${namespace}/imu${imu_suffix}_link</linkName>  <!-- (string, required): name of the body which holds the IMU sensor -->
+         <imuTopic>${imu_topic}</imuTopic>  <!-- (string): name of the sensor output topic and prefix of service names (defaults to imu) -->
+         <gyroscopeNoiseDensity>${gyroscope_noise_density}</gyroscopeNoiseDensity>  <!-- Gyroscope noise density (two-sided spectrum) [rad/s/sqrt(Hz)] -->
+         <gyroscopeRandomWalk>${gyroscopoe_random_walk}</gyroscopeRandomWalk>  <!-- Gyroscope bias random walk [rad/s/s/sqrt(Hz)] -->
+         <gyroscopeBiasCorrelationTime>${gyroscope_bias_correlation_time}</gyroscopeBiasCorrelationTime>  <!-- Gyroscope bias correlation time constant [s] -->
+         <gyroscopeTurnOnBiasSigma>${gyroscope_turn_on_bias_sigma}</gyroscopeTurnOnBiasSigma>  <!-- Gyroscope turn on bias standard deviation [rad/s] -->
+         <accelerometerNoiseDensity>${accelerometer_noise_density}</accelerometerNoiseDensity>  <!-- Accelerometer noise density (two-sided spectrum) [m/s^2/sqrt(Hz)] -->
+         <accelerometerRandomWalk>${accelerometer_random_walk}</accelerometerRandomWalk> <!-- Accelerometer bias random walk. [m/s^2/s/sqrt(Hz)]  -->
+         <accelerometerBiasCorrelationTime>${accelerometer_bias_correlation_time}</accelerometerBiasCorrelationTime> <!-- Accelerometer bias correlation time constant [s]  -->
+         <accelerometerTurnOnBiasSigma>${accelerometer_turn_on_bias_sigma}</accelerometerTurnOnBiasSigma> <!-- Accelerometer turn on bias standard deviation [m/s^2]  -->
+       </plugin>
     </gazebo>
   </xacro:macro>
 <!-- Macro to add a generic odometry sensor. -->
   <xacro:macro name="odometry_plugin_macro"
-    params="
-      namespace odometry_sensor_suffix parent_link pose_topic pose_with_covariance_topic
+    params="namespace odometry_sensor_suffix parent_link pose_topic pose_with_covariance_topic
       position_topic transform_topic odometry_topic parent_frame_id
       mass_odometry_sensor measurement_divisor measurement_delay unknown_delay
@@ -176,5 +176,5 @@
         <mass value="${mass_odometry_sensor}" />  <!-- [kg] -->
       </inertial>
-    </link>
+    </link> -->
     <!-- odometry joint -->
     <joint name="${namespace}/odometry_sensor${odometry_sensor_suffix}_joint" type="revolute">
@@ -184,7 +184,7 @@
       <limit upper="0" lower="0" effort="0" velocity="0" />
     </joint>
-    <gazebo>
-      <plugin filename="librotors_gazebo_odometry_plugin.so" name="odometry_sensor${odometry_sensor_suffix}">
-        <linkName>${namespace}/odometry_sensor${odometry_sensor_suffix}_link</linkName>
+      <gazebo>
+     <plugin filename="librotors_gazebo_odometry_plugin.so" name="odometry_sensor${odometry_sensor_suffix}">
+        <linkName>base_link</linkName>  <!--{namespace}/odometry_sensor${odometry_sensor_suffix}_link"-->
         <robotNamespace>${namespace}</robotNamespace>
         <poseTopic>${pose_topic}</poseTopic>
@@ -194,13 +194,13 @@
         <odometryTopic>${odometry_topic}</odometryTopic>
         <parentFrameId>${parent_frame_id}</parentFrameId>  <!-- Use the scoped link name here. e.g. Model::link. -->
-        <measurementDivisor>${measurement_divisor}</measurementDivisor> <!-- only every (seq % measurementDivisor) == 0 measurement is published [int] -->
-        <measurementDelay>${measurement_delay}</measurementDelay> <!-- time that measurement gets held back before it's published in [simulation cycles (int)] -->
-        <unknownDelay>${unknown_delay}</unknownDelay> <!-- additional delay, that just gets added to the timestamp [s] -->
-        <noiseNormalPosition>${noise_normal_position}</noiseNormalPosition> <!-- standard deviation of additive white gaussian noise [m] -->
-        <noiseNormalQuaternion>${noise_normal_quaternion}</noiseNormalQuaternion> <!-- standard deviation white gaussian noise [rad]: q_m = q*quaternionFromSmallAngleApproximation(noiseNormalQ) -->
-        <noiseNormalLinearVelocity>${noise_normal_linear_velocity}</noiseNormalLinearVelocity> <!-- standard deviation of additive white gaussian noise [m/s] -->
-        <noiseNormalAngularVelocity>${noise_normal_angular_velocity}</noiseNormalAngularVelocity> <!-- standard deviation of additive white gaussian noise [rad/s] -->
-        <noiseUniformPosition>${noise_uniform_position}</noiseUniformPosition> <!-- symmetric bounds of uniform noise [m] -->
-        <noiseUniformQuaternion>${noise_uniform_quaternion}</noiseUniformQuaternion> <!-- symmetric bounds of uniform noise [rad], computation see above -->
+        <measurementDivisor>${measurement_divisor}</measurementDivisor>  <!-- only every (seq % measurementDivisor) == 0 measurement is published [int] -->
+        <measurementDelay>${measurement_delay}</measurementDelay>  <!-- time that measurement gets held back before it's published in [simulation cycles (int)] -->
+        <unknownDelay>${unknown_delay}</unknownDelay>   <!-- additional delay, that just gets added to the timestamp [s] -->
+        <noiseNormalPosition>${noise_normal_position}</noiseNormalPosition>  <!-- standard deviation of additive white gaussian noise [m] -->
+        <noiseNormalQuaternion>${noise_normal_quaternion}</noiseNormalQuaternion>  <!-- standard deviation white gaussian noise [rad]: q_m = q*quaternionFromSmallAngleApproximation(noiseNormalQ) -->
+        <noiseNormalLinearVelocity>${noise_normal_linear_velocity}</noiseNormalLinearVelocity>  <!-- standard deviation of additive white gaussian noise [m/s] -->
+        <noiseNormalAngularVelocity>${noise_normal_angular_velocity}</noiseNormalAngularVelocity>  <!-- standard deviation of additive white gaussian noise [rad/s] -->
+        <noiseUniformPosition>${noise_uniform_position}</noiseUniformPosition>  <!-- symmetric bounds of uniform noise [m] -->
+        <noiseUniformQuaternion>${noise_uniform_quaternion}</noiseUniformQuaternion>  <!-- symmetric bounds of uniform noise [rad], computation see above -->
         <noiseUniformLinearVelocity>${noise_uniform_linear_velocity}</noiseUniformLinearVelocity>  <!-- symmetric bounds of uniform noise [m/s] -->
         <noiseUniformAngularVelocity>${noise_uniform_angular_velocity}</noiseUniformAngularVelocity>  <!-- symmetric bounds of uniform noise [rad/s] -->
@@ -234,5 +234,5 @@
   <!-- VI sensor macros -->
   <!-- Macro to add a VI-sensor camera. -->
-  <xacro:macro name="vi_sensor_camera_macro"
+   <xacro:macro name="vi_sensor_camera_macro"
     params="namespace parent_link camera_suffix frame_rate *origin">
     <xacro:camera_macro
@@ -373,7 +373,7 @@
     </xacro:if>
     <!-- Groundtruth -->
-    <xacro:if value="$(arg enable_ground_truth)">
+   <xacro:if value="$(arg enable_ground_truth)">
       <!-- Odometry Sensor -->
-      <xacro:odometry_plugin_macro
+     <xacro:odometry_plugin_macro
         namespace="${namespace}/ground_truth"
         odometry_sensor_suffix=""
@@ -400,10 +400,10 @@
         odometry_map=""
         image_scale="">
-        <inertia ixx="0.00001" ixy="0.0" ixz="0.0" iyy="0.00001" iyz="0.0" izz="0.00001" /> <!-- [kg.m^2] [kg.m^2] [kg.m^2] [kg.m^2] [kg.m^2] [kg.m^2] -->
-        <origin xyz="0.0 0.0 0.0" rpy="0.0 0.0 0.0" />
+        <inertia ixx="0.00001" ixy="0.0" ixz="0.0" iyy="0.00001" iyz="0.0" izz="0.00001" />  <!-- [kg.m^2] [kg.m^2] [kg.m^2] [kg.m^2] [kg.m^2] [kg.m^2] -->
+      <origin xyz="0.0 0.0 0.0" rpy="0.0 0.0 0.0" />
       </xacro:odometry_plugin_macro>
     </xacro:if>
     <!-- ADIS16448 IMU. -->
-    <xacro:imu_plugin_macro
+     <xacro:imu_plugin_macro
       namespace="${namespace}"
       imu_suffix=""
